Commit message: Change name to gocator interface Add 3520 URDF

File: urdf/GOCATOR-3520.urdf.xacro (robot description, xacro)
@@ -1,9 +1,9 @@
 <?xml version="1.0"?>
-<robot xmlns:xacro="http://www.ros.org/wiki/xacro">
+<robot name="GOCATOR" xmlns:xacro="http://www.ros.org/wiki/xacro">
     <material name="Gocator/Black">
         <color rgba="0.1 0.1 0.1 1.0"/>
     </material>
     <!-- Just the bounding box of the gocator -->
-    <xacro:macro name="gocator_3110" params="parent name">
+    <xacro:macro name="GOCATOR-3520" params="parent name *origin">
         <joint name="${parent}_${name}_anchor" type="fixed">
             <parent link="${parent}" />
@@ -12,16 +12,14 @@
         <link name="${name}">
             <visual>
-                <!-- <origin xyz="0 0 0.05" rpy="0 0 0"/> -->
-                <origin xyz="0 0 0.0623" rpy="3.141592 0 0"/>
+                <origin xyz="0 0 0" rpy="0 0 0"/>
                 <geometry>
-                    <!-- <box size="0.156 0.05 0.1"/> -->
-                    <mesh filename="package://gocator_3100/urdf/gocator_3110.stl" scale="0.001 0.001 0.001"/>
+                    <mesh filename="package://gocator_interface/urdf/GOCATOR-3520.stl" scale="0.001 0.001 0.001"/>
                 </geometry>
                 <material name="Gocator/Black"/>
             </visual>
             <collision>
-                <origin xyz="0 0 0.05" rpy="0 0 0"/>
+                <origin xyz="0 0 0" rpy="0 0 0"/>
                 <geometry>
-                    <box size="0.310 0.10 0.1"/>
+                    <mesh filename="package://gocator_interface/urdf/GOCATOR-3520.stl" scale="0.001 0.001 0.001"/>
                 </geometry>
             </collision>
@@ -30,5 +28,5 @@
             <parent link="${name}"/>
             <child link="${name}_point_cloud"/>
-            <origin xyz="0 0 ${0.0623+0.150+0.05}" rpy="0 3.141592 -1.570796"/>  <!--27.9cm from parent -->
+            <origin xyz="0 0 0.167" rpy="0 0 0"/>
         </joint>
         <link name="${name}_point_cloud"/>
@@ -37,3 +35,7 @@
         </gazebo>
     </xacro:macro>
+   <link name="world" />
+  <xacro:GOCATOR-3520 parent="world" name="gocator">
+    <origin xyz="0.0 0.0 0.0" rpy="0 0 0"/>
+  </xacro:GOCATOR-3520>
 </robot>

Commit message: Tested with real camera and ROS toppic.

File: urdf/GOCATOR-3520.urdf.xacro (robot description, xacro)
@@ -8,7 +8,7 @@
         <joint name="${parent}_${name}_anchor" type="fixed">
             <parent link="${parent}" />
-            <child link="${name}" />
+            <child link="${name}_link" />
         </joint>
-        <link name="${name}">
+        <link name="${name}_link">
             <visual>
                 <origin xyz="0 0 0" rpy="0 0 0"/>
@@ -26,16 +26,12 @@
         </link>
         <joint name="${name}_point_cloud_anchor" type="fixed" >
-            <parent link="${name}"/>
+            <parent link="${name}_link"/>
             <child link="${name}_point_cloud"/>
-            <origin xyz="0 0 0.167" rpy="0 0 0"/>
+            <origin xyz="0 0 ${0.075+0.203+0.167}" rpy="3.141592 0 1.570796"/>
         </joint>
         <link name="${name}_point_cloud"/>
-        <gazebo reference="${name}">
+        <gazebo reference="GOCATOR-3520">
             <static>true</static>
         </gazebo>
     </xacro:macro>
-   <link name="world" />
-  <xacro:GOCATOR-3520 parent="world" name="gocator">
-    <origin xyz="0.0 0.0 0.0" rpy="0 0 0"/>
-  </xacro:GOCATOR-3520>
 </robot>
